File: пред/preamp.kicad_pcb (KiCad board)
At the start: 2 copper layers, 48 parts, among them P1 CONN_01X02, P2 CONN_01X03, P3 CONN_01X03, P4 CONN_01X03, P5 CONN_01X02, P6 CONN_01X02, P7 CONN_01X03, Q1 BSS138, Q2 BSS138, Q3 BC857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

Commit message: Начата трассировка
Parts:
- moved C9 96.7 mm to (179.0, 43.8), turned to 90 degrees
- moved P4 81.3 mm to (147.5, 51.0), turned to 270 degrees
- moved R24 78.1 mm to (182.5, 41.5), turned to 90 degrees
- moved R23 71.6 mm to (182.2, 51.0), turned to 270 degrees
- moved P3 70.5 mm to (138.2, 48.0)
- moved R1 70.5 mm to (134.4, 36.2)
- moved R18 69.1 mm to (164.2, 49.2), turned to 270 degrees
- moved C5 69.0 mm to (172.2, 45.2), turned to 270 degrees
- moved C1 66.3 mm to (112.8, 43.8)
- moved Q5 65.1 mm to (168.0, 50.0)
- moved Q1 63.7 mm to (124.2, 43.5)
- moved Q4 62.3 mm to (163.3, 53.5), turned to 90 degrees
- moved Q6 61.9 mm to (168.0, 41.5)
- moved R19 61.5 mm to (164.2, 44.5), turned to 270 degrees
- moved R16 60.1 mm to (171.3, 39.0)
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Connections:
- Q6 pad 3: Net-(Q6-Pad3) -> Net-(C9-Pad2)
Routing:
- net Net-(C8-Pad2): track 0.00 -> 16.6 mm
- net Net-(C9-Pad2): track 0.00 -> 15.5 mm
- net Net-(C5-Pad2): track 0.00 -> 14.1 mm
- net GNDREF: track 0.00 -> 12.8 mm
- net Net-(C5-Pad1): track 0.00 -> 11.3 mm
- net Net-(C4-Pad1): track 0.00 -> 10.4 mm
- net Net-(C4-Pad2): track 0.00 -> 8.79 mm
- net Net-(C6-Pad2): track 0.00 -> 6.91 mm
- net Net-(P2-Pad1): track 0.00 -> 6.27 mm
- net Net-(C7-Pad1): track 0.00 -> 5.24 mm
- net Net-(P7-Pad1): track 0.00 -> 4.23 mm
- net Net-(P7-Pad3): track 0.00 -> 4.19 mm
- net Net-(Q3-Pad2): track 0.00 -> 3.12 mm
- net Net-(Q6-Pad2): track 0.00 -> 3.04 mm
- net Net-(Q5-Pad2): track 0.00 -> 2.96 mm
