File: пред/preamp-cp/preamp (копия).sch (KiCad schematic (older format))
At the start: 48 parts, among them P1 CONN_01X02, P2 CONN_01X03, P3 CONN_01X03, P4 CONN_01X03, P5 CONN_01X02, P6 CONN_01X02, P7 CONN_01X03, Q1 BSS138, Q2 BSS138, Q3 BC857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

Commit message: add new board for preamp
Parts:
- C1, C4: value C -> 0.15u; footprint Capacitors_SMD:C_0805 -> Capacitors_THT:C_Rect_L7.2mm_W2.5mm_P5.00mm_FKS2_FKP2_MKS2_MKP2
- C10: value C -> 0.01u; footprint Capacitors_SMD:C_0805 -> Capacitors_THT:C_Rect_L7.2mm_W2.5mm_P5.00mm_FKS2_FKP2_MKS2_MKP2
- C2, C5: value C -> 0.1u; footprint Capacitors_SMD:C_0805 -> Capacitors_THT:C_Rect_L7.2mm_W2.5mm_P5.00mm_FKS2_FKP2_MKS2_MKP2
- C3: value C -> 0.015u; footprint Capacitors_SMD:C_0805 -> Capacitors_THT:C_Rect_L7.2mm_W2.5mm_P5.00mm_FKS2_FKP2_MKS2_MKP2
- C6: value C -> 0.047u; footprint Capacitors_SMD:C_0805 -> Capacitors_THT:C_Rect_L7.2mm_W2.5mm_P5.00mm_FKS2_FKP2_MKS2_MKP2
- C7: value C -> 3300p; footprint Capacitors_SMD:C_0805 -> Capacitors_THT:C_Rect_L7.2mm_W2.5mm_P5.00mm_FKS2_FKP2_MKS2_MKP2
- C8, C9: value C -> 5u
- P1, P5, P6: footprint Pin_Headers:Pin_Header_Angled_1x02_Pitch2.54mm -> Pin_Headers:Pin_Header_Straight_1x02_Pitch2.54mm; symbol CONN_01X02 -> Conn_01x02
- P2, P7: symbol CONN_01X03 -> Conn_01x03
- R1: value R -> 4.7M
- R10, R16: value R -> 18k
- R11, R17: value R -> 470R
- R12: value R -> 2k2
- R13: value R -> 680R
- R14: value R -> 2k1
- R15: value R -> 180R
- R18, R19: value R -> 33R
- R2, R6: value R -> 12k
- R20: value R -> 8k2
- R21: value R -> 2k
- R22: value R -> 2M2
- R23, R24: value R -> 1k2
- R25: renamed from P4; value CONN_01X03 -> 100k; symbol CONN_01X03 -> Conn_01x03
- R26: renamed from P3; value CONN_01X03 -> 100k; symbol CONN_01X03 -> Conn_01x03
- R3: value R -> 8.48k
- R4: value R -> 1k
- R5: value R -> 22k
- R7: value R -> 22.1k
- R8: value R -> 68.1k
- R9: value R -> 2.2M
- RV1: value POT -> 2k2; footprint Potentiometers:Potentiometer_Trimmer_Bourns_3299W -> Potentiometers:Potentiometer_Trimmer_Bourns_3296W
Connections:
- wire segments 112 -> 115
Other:
- moved on the sheet: C1

Commit message: Переделана печатная плата преда
Parts:
- C6: footprint Capacitors_THT:C_Rect_L7.2mm_W2.5mm_P5.00mm_FKS2_FKP2_MKS2_MKP2 -> Capacitors_THT:C_Rect_L11.5mm_W5.0mm_P10.00mm_MKT
Changed lines of the file:
@@
 LIBS:contrib
 LIBS:valves
+LIBS:74xgxx
+LIBS:ac-dc
+LIBS:actel
+LIBS:allegro
+LIBS:Altera
+LIBS:analog_devices
+LIBS:battery_management
+LIBS:bbd
+LIBS:bosch
+LIBS:brooktre
+LIBS:cmos_ieee
+LIBS:dc-dc
+LIBS:diode
+LIBS:elec-unifil
+LIBS:ESD_Protection
+LIBS:ftdi
+LIBS:gennum
+LIBS:graphic_symbols
+LIBS:hc11
+LIBS:infineon
+LIBS:intersil
+LIBS:ir
+LIBS:Lattice
+LIBS:leds
+LIBS:LEM
+LIBS:logic_programmable
+LIBS:maxim
+LIBS:mechanical
+LIBS:microchip_dspic33dsc
+LIBS:microchip_pic10mcu
+LIBS:microchip_pic12mcu
+LIBS:microchip_pic16mcu
+LIBS:microchip_pic18mcu
+LIBS:microchip_pic24mcu
+LIBS:microchip_pic32mcu
+LIBS:modules
+LIBS:motor_drivers
+LIBS:msp430
+LIBS:nordicsemi
+LIBS:nxp
+LIBS:nxp_armmcu
+LIBS:onsemi
+LIBS:Oscillators
+LIBS:powerint
+LIBS:Power_Management
+LIBS:pspice
+LIBS:references
+LIBS:rfcom
+LIBS:RFSolutions
+LIBS:sensors
+LIBS:silabs
+LIBS:stm8
+LIBS:stm32
+LIBS:supertex
+LIBS:transf
+LIBS:triac_thyristor
+LIBS:ttl_ieee
+LIBS:video
+LIBS:wiznet
+LIBS:Worldsemi
+LIBS:Xicor
+LIBS:zetex
+LIBS:Zilog
 LIBS:preamp (копия)-cache
 EELAYER 25 0
@@
 F 0 "C6" H 7400 4850 50  0000 C CNN
 F 1 "0.047u" H 7400 4950 50  0000 C CNN
-F 2 "Capacitors_THT:C_Rect_L7.2mm_W2.5mm_P5.00mm_FKS2_FKP2_MKS2_MKP2" H 7250 4850 50  0001 C CNN
+F 2 "Capacitors_THT:C_Rect_L11.5mm_W5.0mm_P10.00mm_MKT" H 7250 4850 50  0001 C CNN
 F 3 "" H 7250 4850 50  0000 C CNN
 	1    7250 4850
