File: стабилизатор/Стабилизатор.sch (KiCad schematic (older format))
At the start: 35 parts, among them J1 V_IN, J2 +43V, J3 -43V, J4 +11V, J5 -11V, J6 +31V, J7 -31V, J8 V_OUT, Q1 BD140, Q2 BD139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

Commit message: Привязка корпусов
Parts:
- C1, C2, C4, C5, C6, C7: footprint (none) -> Capacitors_THT:CP_Radial_D5.0mm_P2.50mm
- C3: footprint (none) -> Capacitors_SMD:C_0805_HandSoldering
- D1, D2: footprint (none) -> Diodes_THT:D_DO-35_SOD27_P7.62mm_Horizontal
- J1, J8: footprint (none) -> Pin_Headers:Pin_Header_Straight_1x03_Pitch2.54mm
- J2, J3, J4, J5, J6, J7: footprint (none) -> Measurement_Points:Measurement_Point_Round-SMD-Pad_Small
- R1, R10, R11, R12, R2, R3, R4, R5, R6, R7, R8, R9: footprint (none) -> Resistors_SMD:R_1206_HandSoldering
- RV1, RV2: footprint (none) -> Potentiometers:Potentiometer_Trimmer_Bourns_3266Y
Changed lines of the file:
@@
 F 0 "C3" H 5350 1800 50  0000 L CNN
 F 1 "120nF" H 5350 1700 50  0000 L CNN
-F 2 "" H 5238 1600 50  0001 C CNN
+F 2 "Capacitors_SMD:C_0805_HandSoldering" H 5238 1600 50  0001 C CNN
 F 3 "" H 5200 1750 50  0001 C CNN
 	1    5200 1750
@@
 F 0 "R8" V 4150 1450 50  0000 C CNN
 F 1 "10R" V 4250 1500 50  0000 C CNN
-F 2 "" V 4280 1500 50  0001 C CNN
+F 2 "Resistors_SMD:R_1206_HandSoldering" V 4280 1500 50  0001 C CNN
 F 3 "" H 4350 1500 50  0001 C CNN
 	1    4350 1500
@@
 F 0 "R5" H 4000 1750 50  0000 C CNN
 F 1 "1k" H 3950 1850 50  0000 C CNN
-F 2 "" V 4030 1750 50  0001 C CNN
+F 2 "Resistors_SMD:R_1206_HandSoldering" V 4030 1750 50  0001 C CNN
 F 3 "" H 4100 1750 50  0001 C CNN
 	1    4100 1750
@@
 F 0 "D2" V 5700 1900 50  0000 C CNN
 F 1 "20V" V 5800 1900 50  0000 C CNN
-F 2 "" H 5700 1750 50  0001 C CNN
+F 2 "Diodes_THT:D_DO-35_SOD27_P7.62mm_Horizontal" H 5700 1750 50  0001 C CNN
 F 3 "" H 5700 1750 50  0001 C CNN
 	1    5700 1750
@@
 F 0 "R9" H 6050 1850 50  0000 C CNN
 F 1 "18k" H 6050 1950 50  0000 C CNN
-F 2 "" V 6130 1850 50  0001 C CNN
+F 2 "Resistors_SMD:R_1206_HandSoldering" V 6130 1850 50  0001 C CNN
 F 3 "" H 6200 1850 50  0001 C CNN
 	1    6200 1850
@@
 F 0 "RV1" H 6050 2250 50  0000 C CNN
 F 1 "4k7" H 6050 2350 50  0000 C CNN
-F 2 "" H 6200 2300 50  0001 C CNN
+F 2 "Potentiometers:Potentiometer_Trimmer_Bourns_3266Y" H 6200 2300 50  0001 C CNN
 F 3 "" H 6200 2300 50  0001 C CNN
 	1    6200 2300
@@
 F 0 "R10" H 6050 2700 50  0000 C CNN
 F 1 "12k" H 6050 2800 50  0000 C CNN
-F 2 "" V 6130 2700 50  0001 C CNN
+F 2 "Resistors_SMD:R_1206_HandSoldering" V 6130 2700 50  0001 C CNN
 F 3 "" H 6200 2700 50  0001 C CNN
 	1    6200 2700
@@
 F 0 "R1" H 3300 1750 50  0000 C CNN
 F 1 "6k2" H 3250 1850 50  0000 C CNN
-F 2 "" V 3330 1750 50  0001 C CNN
+F 2 "Resistors_SMD:R_1206_HandSoldering" V 3330 1750 50  0001 C CNN
 F 3 "" H 3400 1750 50  0001 C CNN
 	1    3400 1750
@@
 F 0 "R3" V 3500 2150 50  0000 C CNN
 F 1 "5k6" V 3600 2200 50  0000 C CNN
-F 2 "" V 3630 2200 50  0001 C CNN
+F 2 "Resistors_SMD:R_1206_HandSoldering" V 3630 2200 50  0001 C CNN
 F 3 "" H 3700 2200 50  0001 C CNN
 	1    3700 2200
@@
 F 0 "C1" H 3450 2300 50  0000 L CNN
 F 1 "5uF" H 3450 2200 50  0000 L CNN
-F 2 "" H 3438 2300 50  0001 C CNN
+F 2 "Capacitors_THT:CP_Radial_D5.0mm_P2.50mm" H 3438 2300 50  0001 C CNN
 F 3 "" H 3400 2450 50  0001 C CNN
 	1    3400 2450
@@
 F 0 "C4" H 5875 2650 50  0000 L CNN
 F 1 "5uF" H 5875 2450 50  0000 L CNN
-F 2 "" H 5888 2400 50  0001 C CNN
+F 2 "Capacitors_THT:CP_Radial_D5.0mm_P2.50mm" H 5888 2400 50  0001 C CNN
 F 3 "" H 5850 2550 50  0001 C CNN
 	1    5850 2550
@@
 F 0 "C6" H 6750 2050 50  0000 L CNN
 F 1 "5uF" H 6750 1950 50  0000 L CNN
-F 2 "" H 6688 2000 50  0001 C CNN
+F 2 "Capacitors_THT:CP_Radial_D5.0mm_P2.50mm" H 6688 2000 50  0001 C CNN
 F 3 "" H 6650 2150 50  0001 C CNN
 	1    6650 2150
@@
 F 0 "R4" V 3500 3850 50  0000 C CNN
 F 1 "5k6" V 3600 3900 50  0000 C CNN
-F 2 "" V 3630 3700 50  0001 C CNN
+F 2 "Resistors_SMD:R_1206_HandSoldering" V 3630 3700 50  0001 C CNN
 F 3 "" H 3700 3700 50  0001 C CNN
 	1    3700 3700
@@
 F 0 "R2" H 3300 3900 50  0000 C CNN
 F 1 "6k2" H 3250 4000 50  0000 C CNN
-F 2 "" V 3330 3900 50  0001 C CNN
+F 2 "Resistors_SMD:R_1206_HandSoldering" V 3330 3900 50  0001 C CNN
 F 3 "" H 3400 3900 50  0001 C CNN
 	1    3400 3900
@@
 F 0 "C2" H 3450 3150 50  0000 L CNN
 F 1 "5uF" H 3450 3050 50  0000 L CNN
-F 2 "" H 3438 3150 50  0001 C CNN
+F 2 "Capacitors_THT:CP_Radial_D5.0mm_P2.50mm" H 3438 3150 50  0001 C CNN
 F 3 "" H 3400 3300 50  0001 C CNN
 	1    3400 3300
@@
 F 0 "R6" H 4000 4050 50  0000 C CNN
 F 1 "1k" H 4000 4150 50  0000 C CNN
-F 2 "" V 4030 4200 50  0001 C CNN
+F 2 "Resistors_SMD:R_1206_HandSoldering" V 4030 4200 50  0001 C CNN
 F 3 "" H 4100 4200 50  0001 C CNN
 	1    4100 4200
@@
 F 0 "R7" V 4100 4550 50  0000 C CNN
 F 1 "10R" V 4200 4550 50  0000 C CNN
-F 2 "" V 4230 4400 50  0001 C CNN
+F 2 "Resistors_SMD:R_1206_HandSoldering" V 4230 4400 50  0001 C CNN
 F 3 "" H 4300 4400 50  0001 C CNN
 	1    4300 4400
@@
 F 0 "C5" H 5875 3450 50  0000 L CNN
 F 1 "5uF" H 5875 3250 50  0000 L CNN
-F 2 "" H 5888 3200 50  0001 C CNN
+F 2 "Capacitors_THT:CP_Radial_D5.0mm_P2.50mm" H 5888 3200 50  0001 C CNN
 F 3 "" H 5850 3350 50  0001 C CNN
 	1    5850 3350
@@
 F 0 "R11" H 6100 3350 50  0000 C CNN
 F 1 "12k" H 6050 3450 50  0000 C CNN
-F 2 "" V 6130 3350 50  0001 C CNN
+F 2 "Resistors_SMD:R_1206_HandSoldering" V 6130 3350 50  0001 C CNN
 F 3 "" H 6200 3350 50  0001 C CNN
 	1    6200 3350
@@
 F 0 "RV2" H 6050 3700 50  0000 C CNN
 F 1 "4k7" H 6050 3800 50  0000 C CNN
-F 2 "" H 6200 3750 50  0001 C CNN
+F 2 "Potentiometers:Potentiometer_Trimmer_Bourns_3266Y" H 6200 3750 50  0001 C CNN
 F 3 "" H 6200 3750 50  0001 C CNN
 	1    6200 3750
@@
 F 0 "D1" V 5450 4150 50  0000 C CNN
 F 1 "20V" V 5550 4150 50  0000 C CNN
-F 2 "" H 5450 4000 50  0001 C CNN
+F 2 "Diodes_THT:D_DO-35_SOD27_P7.62mm_Horizontal" H 5450 4000 50  0001 C CNN
 F 3 "" H 5450 4000 50  0001 C CNN
 	1    5450 4000
@@
 F 0 "C7" H 6750 3600 50  0000 L CNN
 F 1 "5uF" H 6750 3500 50  0000 L CNN
-F 2 "" H 6688 3600 50  0001 C CNN
+F 2 "Capacitors_THT:CP_Radial_D5.0mm_P2.50mm" H 6688 3600 50  0001 C CNN
 F 3 "" H 6650 3750 50  0001 C CNN
 	1    6650 3750
@@
 F 0 "R12" H 6350 4100 50  0000 C CNN
 F 1 "18k" H 6350 4200 50  0000 C CNN
-F 2 "" V 6130 4150 50  0001 C CNN
+F 2 "Resistors_SMD:R_1206_HandSoldering" V 6130 4150 50  0001 C CNN
 F 3 "" H 6200 4150 50  0001 C CNN
 	1    6200 4150
@@
 F 0 "J5" H 5300 3450 50  0000 C CNN
 F 1 "-11V" H 5300 3350 50  0000 C CNN
-F 2 "" H 5650 3350 50  0001 C CNN
+F 2 "Measurement_Points:Measurement_Point_Round-SMD-Pad_Small" H 5650 3350 50  0001 C CNN
 F 3 "" H 5650 3350 50  0001 C CNN
 	1    5450 3350
@@
 F 0 "J4" H 5550 2700 50  0000 C CNN
 F 1 "+11V" H 5600 2800 50  0000 C CNN
-F 2 "" H 5650 2650 50  0001 C CNN
+F 2 "Measurement_Points:Measurement_Point_Round-SMD-Pad_Small" H 5650 2650 50  0001 C CNN
 F 3 "" H 5650 2650 50  0001 C CNN
 	1    5450 2650
@@
 F 0 "J2" H 3650 1550 50  0000 C CNN
 F 1 "+43V" H 3600 1650 50  0000 C CNN
-F 2 "" H 3950 1550 50  0001 C CNN
+F 2 "Measurement_Points:Measurement_Point_Round-SMD-Pad_Small" H 3950 1550 50  0001 C CNN
 F 3 "" H 3950 1550 50  0001 C CNN
 	1    3750 1550
@@
 F 0 "J3" H 3700 4450 50  0000 C CNN
 F 1 "-43V" H 3700 4350 50  0000 C CNN
-F 2 "" H 4050 4350 50  0001 C CNN
+F 2 "Measurement_Points:Measurement_Point_Round-SMD-Pad_Small" H 4050 4350 50  0001 C CNN
 F 3 "" H 4050 4350 50  0001 C CNN
 	1    3850 4350
@@
 F 0 "J7" H 6400 4400 50  0000 C CNN
 F 1 "-31V" H 6400 4300 50  0000 C CNN
-F 2 "" H 6750 4300 50  0001 C CNN
+F 2 "Measurement_Points:Measurement_Point_Round-SMD-Pad_Small" H 6750 4300 50  0001 C CNN
 F 3 "" H 6750 4300 50  0001 C CNN
 	1    6550 4300
@@
 F 0 "J6" H 6200 1550 50  0000 C CNN
 F 1 "+31V" H 6150 1650 50  0000 C CNN
-F 2 "" H 6500 1550 50  0001 C CNN
+F 2 "Measurement_Points:Measurement_Point_Round-SMD-Pad_Small" H 6500 1550 50  0001 C CNN
 F 3 "" H 6500 1550 50  0001 C CNN
 	1    6300 1550
@@
 F 0 "J1" H 2750 3200 50  0000 C CNN
 F 1 "V_IN" H 2750 2800 50  0000 C CNN
-F 2 "" H 2750 3000 50  0001 C CNN
+F 2 "Pin_Headers:Pin_Header_Straight_1x03_Pitch2.54mm" H 2750 3000 50  0001 C CNN
 F 3 "" H 2750 3000 50  0001 C CNN
 	1    2750 3000
@@
 F 0 "J8" H 7250 3200 50  0000 C CNN
 F 1 "V_OUT" H 7250 2800 50  0000 C CNN
-F 2 "" H 7250 3000 50  0001 C CNN
+F 2 "Pin_Headers:Pin_Header_Straight_1x03_Pitch2.54mm" H 7250 3000 50  0001 C CNN
 F 3 "" H 7250 3000 50  0001 C CNN
 	1    7250 3000

Commit message: Разводка платы стабилизатора
Parts:
- Q3, Q4: footprint TO_SOT_Packages_THT:TO-92_Molded_Narrow -> TO_SOT_Packages_THT:TO-92_Molded_Wide
Changed lines of the file:
@@
 F 0 "Q4" H 4800 3550 50  0000 L CNN
 F 1 "2N3905" H 4600 3650 50  0000 L CNN
-F 2 "TO_SOT_Packages_THT:TO-92_Molded_Narrow" H 5150 3675 50  0001 L CIN
+F 2 "TO_SOT_Packages_THT:TO-92_Molded_Wide" H 5150 3675 50  0001 L CIN
 F 3 "" H 4950 3750 50  0001 L CNN
 	1    4950 3750
@@
 F 0 "Q3" H 4750 2500 50  0000 L CNN
 F 1 "2N3904" H 4550 2400 50  0000 L CNN
-F 2 "TO_SOT_Packages_THT:TO-92_Molded_Narrow" H 5150 2225 50  0001 L CIN
+F 2 "TO_SOT_Packages_THT:TO-92_Molded_Wide" H 5150 2225 50  0001 L CIN
 F 3 "" H 4950 2300 50  0001 L CNN
 	1    4950 2300
