File: preamp-comby/Power.sch (KiCad schematic (older format))
At the start: 35 parts, among them J201 Screw_Terminal_01x03, Q201 BD140, Q202 BD139, Q203 2N3904, Q204 2N3905

Commit message: Finish schematic, start routing
Parts:
- C201, C202, C205, C206, C207, C208: footprint (none) -> Capacitor_THT:CP_Radial_D5.0mm_P2.00mm
- C203, C204: footprint (none) -> Capacitor_THT:C_Rect_L7.2mm_W3.0mm_P5.00mm_FKS2_FKP2_MKS2_MKP2
Changed lines of the file:
@@
 EESchema Schematic File Version 4
+LIBS:Hierarchy-cache
 EELAYER 30 0
 EELAYER END
@@
 F 0 "C204" H 5900 4950 50  0000 L CNN
 F 1 "120n" H 5900 4750 50  0000 L CNN
-F 2 "" H 6138 4700 50  0001 C CNN
+F 2 "Capacitor_THT:C_Rect_L7.2mm_W3.0mm_P5.00mm_FKS2_FKP2_MKS2_MKP2" H 6138 4700 50  0001 C CNN
 F 3 "~" H 6100 4850 50  0001 C CNN
 	1    6100 4850
@@
 F 0 "C202" H 4518 4146 50  0000 L CNN
 F 1 "5uF" H 4518 4055 50  0000 L CNN
-F 2 "" H 4438 3950 50  0001 C CNN
+F 2 "Capacitor_THT:CP_Radial_D5.0mm_P2.00mm" H 4438 3950 50  0001 C CNN
 F 3 "~" H 4400 4100 50  0001 C CNN
 	1    4400 4100
@@
 F 0 "C201" H 4518 3646 50  0000 L CNN
 F 1 "5uF" H 4518 3555 50  0000 L CNN
-F 2 "" H 4438 3450 50  0001 C CNN
+F 2 "Capacitor_THT:CP_Radial_D5.0mm_P2.00mm" H 4438 3450 50  0001 C CNN
 F 3 "~" H 4400 3600 50  0001 C CNN
 	1    4400 3600
@@
 F 0 "C203" H 5800 2800 50  0000 L CNN
 F 1 "120nF" H 5800 2700 50  0000 L CNN
-F 2 "" H 6138 2700 50  0001 C CNN
+F 2 "Capacitor_THT:C_Rect_L7.2mm_W3.0mm_P5.00mm_FKS2_FKP2_MKS2_MKP2" H 6138 2700 50  0001 C CNN
 F 3 "~" H 6100 2850 50  0001 C CNN
 	1    6100 2850
@@
 F 0 "C207" H 7268 3346 50  0000 L CNN
 F 1 "5uF" H 7268 3255 50  0000 L CNN
-F 2 "" H 7188 3150 50  0001 C CNN
+F 2 "Capacitor_THT:CP_Radial_D5.0mm_P2.00mm" H 7188 3150 50  0001 C CNN
 F 3 "~" H 7150 3300 50  0001 C CNN
 	1    7150 3300
@@
 F 0 "C205" H 6200 3650 50  0000 L CNN
 F 1 "5uF" H 6250 3550 50  0000 L CNN
-F 2 "" H 6538 3500 50  0001 C CNN
+F 2 "Capacitor_THT:CP_Radial_D5.0mm_P2.00mm" H 6538 3500 50  0001 C CNN
 F 3 "~" H 6500 3650 50  0001 C CNN
 	1    6500 3650
@@
 F 0 "C208" H 7268 4446 50  0000 L CNN
 F 1 "5uF" H 7268 4355 50  0000 L CNN
-F 2 "" H 7188 4250 50  0001 C CNN
+F 2 "Capacitor_THT:CP_Radial_D5.0mm_P2.00mm" H 7188 4250 50  0001 C CNN
 F 3 "~" H 7150 4400 50  0001 C CNN
 	1    7150 4400
@@
 F 0 "C206" H 6250 4300 50  0000 L CNN
 F 1 "5uF" H 6250 4200 50  0000 L CNN
-F 2 "" H 6538 3950 50  0001 C CNN
+F 2 "Capacitor_THT:CP_Radial_D5.0mm_P2.00mm" H 6538 3950 50  0001 C CNN
 F 3 "~" H 6500 4100 50  0001 C CNN
 	1    6500 4100
