File: preamp-comby/Preamp.sch (KiCad schematic (older format))
At the start: 47 parts, among them J301 Tone block On/Off, J302 100k, J303 IN, J304 100k, J305 OUT, J306 9K Filter On/Off, Q301 BSS138, Q302 BSS138, Q303 BC850, Q304 BC850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

Commit message: Finish schematic, start routing
Parts:
- C301, C302, C303, C304, C305, C306, C309, C310: footprint (none) -> Capacitor_THT:C_Rect_L7.2mm_W3.0mm_P5.00mm_FKS2_FKP2_MKS2_MKP2
- C307, C308: footprint (none) -> Capacitor_THT:CP_Radial_D5.0mm_P2.00mm
Changed lines of the file:
@@
 EESchema Schematic File Version 4
+LIBS:Hierarchy-cache
 EELAYER 30 0
 EELAYER END
@@
 F 0 "C309" H 7765 2396 50  0000 L CNN
 F 1 "0.1u" H 7765 2305 50  0000 L CNN
-F 2 "" H 7688 2200 50  0001 C CNN
+F 2 "Capacitor_THT:C_Rect_L7.2mm_W3.0mm_P5.00mm_FKS2_FKP2_MKS2_MKP2" H 7688 2200 50  0001 C CNN
 F 3 "~" H 7650 2350 50  0001 C CNN
 	1    7650 2350
@@
 F 0 "C304" V 3998 2400 50  0000 C CNN
 F 1 "0.15u" V 4089 2400 50  0000 C CNN
-F 2 "" H 4288 2250 50  0001 C CNN
+F 2 "Capacitor_THT:C_Rect_L7.2mm_W3.0mm_P5.00mm_FKS2_FKP2_MKS2_MKP2" H 4288 2250 50  0001 C CNN
 F 3 "~" H 4250 2400 50  0001 C CNN
 	1    4250 2400
@@
 F 0 "C310" H 9350 2650 50  0000 R CNN
 F 1 "0.01u" H 9350 2750 50  0000 R CNN
-F 2 "" H 9088 2450 50  0001 C CNN
+F 2 "Capacitor_THT:C_Rect_L7.2mm_W3.0mm_P5.00mm_FKS2_FKP2_MKS2_MKP2" H 9088 2450 50  0001 C CNN
 F 3 "~" H 9050 2600 50  0001 C CNN
 	1    9050 2600
@@
 	1    0    0    -1
 $EndComp
-$Comp
-L power:GNDA #PWR0310
-U 1 1 5D9DE517
-P 9300 2550
-F 0 "#PWR0310" H 9300 2300 50  0001 C CNN
-F 1 "GNDA" H 9305 2377 50  0001 C CNN
-F 2 "" H 9300 2550 50  0001 C CNN
-F 3 "" H 9300 2550 50  0001 C CNN
-	1    9300 2550
-	1    0    0    -1
-$EndComp
 Wire Wire Line
 	9400 2450 9300 2450
@@
 F 0 "C308" H 7182 3654 50  0000 R CNN
 F 1 "5u" H 7182 3745 50  0000 R CNN
-F 2 "" H 7338 3550 50  0001 C CNN
+F 2 "Capacitor_THT:CP_Radial_D5.0mm_P2.00mm" H 7338 3550 50  0001 C CNN
 F 3 "~" H 7300 3700 50  0001 C CNN
 	1    7300 3700
@@
 F 0 "C307" H 7418 1346 50  0000 L CNN
 F 1 "5u" H 7418 1255 50  0000 L CNN
-F 2 "" H 7338 1150 50  0001 C CNN
+F 2 "Capacitor_THT:CP_Radial_D5.0mm_P2.00mm" H 7338 1150 50  0001 C CNN
 F 3 "~" H 7300 1300 50  0001 C CNN
 	1    7300 1300
@@
 F 0 "C302" H 3015 4046 50  0000 L CNN
 F 1 "0,1u" H 3015 3955 50  0000 L CNN
-F 2 "" H 2938 3850 50  0001 C CNN
+F 2 "Capacitor_THT:C_Rect_L7.2mm_W3.0mm_P5.00mm_FKS2_FKP2_MKS2_MKP2" H 2938 3850 50  0001 C CNN
 F 3 "~" H 2900 4000 50  0001 C CNN
 	1    2900 4000
@@
 F 0 "C303" H 4200 5750 50  0000 L CNN
 F 1 "0.15u" H 4200 5550 50  0000 L CNN
-F 2 "" H 4188 5500 50  0001 C CNN
+F 2 "Capacitor_THT:C_Rect_L7.2mm_W3.0mm_P5.00mm_FKS2_FKP2_MKS2_MKP2" H 4188 5500 50  0001 C CNN
 F 3 "~" H 4150 5650 50  0001 C CNN
 	1    4150 5650
@@
 F 0 "C306" H 5200 5750 50  0000 L CNN
 F 1 "0.047u" H 5200 5550 50  0000 L CNN
-F 2 "" H 5188 5500 50  0001 C CNN
+F 2 "Capacitor_THT:C_Rect_L7.2mm_W3.0mm_P5.00mm_FKS2_FKP2_MKS2_MKP2" H 5188 5500 50  0001 C CNN
 F 3 "~" H 5150 5650 50  0001 C CNN
 	1    5150 5650
@@
 F 0 "C301" H 2965 6496 50  0000 L CNN
 F 1 "0.015u" H 2965 6405 50  0000 L CNN
-F 2 "" H 2888 6300 50  0001 C CNN
+F 2 "Capacitor_THT:C_Rect_L7.2mm_W3.0mm_P5.00mm_FKS2_FKP2_MKS2_MKP2" H 2888 6300 50  0001 C CNN
 F 3 "~" H 2850 6450 50  0001 C CNN
 	1    2850 6450
@@
 F 0 "C305" V 4800 6350 50  0000 C CNN
 F 1 "3300p" V 4950 6350 50  0000 C CNN
-F 2 "" H 4888 6000 50  0001 C CNN
+F 2 "Capacitor_THT:C_Rect_L7.2mm_W3.0mm_P5.00mm_FKS2_FKP2_MKS2_MKP2" H 4888 6000 50  0001 C CNN
 F 3 "~" H 4850 6150 50  0001 C CNN
 	1    4850 6150
@@
 	6350 4750 5800 4750
 Connection ~ 5800 4750
+Text HLabel 1800 1750 0    50   Input ~ 0
+GND
+$Comp
+L power:GNDPWR #PWR0101
+U 1 1 5DA39738
+P 1900 1900
+F 0 "#PWR0101" H 1900 1700 50  0001 C CNN
+F 1 "GNDPWR" H 1904 1746 50  0001 C CNN
+F 2 "" H 1900 1850 50  0001 C CNN
+F 3 "" H 1900 1850 50  0001 C CNN
+	1    1900 1900
+	1    0    0    -1
+$EndComp
+$Comp
+L power:GNDA #PWR0102
+U 1 1 5DA3BFD3
+P 1850 2400
+F 0 "#PWR0102" H 1850 2150 50  0001 C CNN
+F 1 "GNDA" H 1855 2227 50  0001 C CNN
+F 2 "" H 1850 2400 50  0001 C CNN
+F 3 "" H 1850 2400 50  0001 C CNN
+	1    1850 2400
+	1    0    0    -1
+$EndComp
+Wire Wire Line
+	1800 1750 1900 1750
+Wire Wire Line
+	1900 1750 1900 1900
+$Comp
+L power:GNDPWR #PWR0103
+U 1 1 5DA47103
+P 9300 2550
+F 0 "#PWR0103" H 9300 2350 50  0001 C CNN
+F 1 "GNDPWR" H 9304 2396 50  0001 C CNN
+F 2 "" H 9300 2500 50  0001 C CNN
+F 3 "" H 9300 2500 50  0001 C CNN
+	1    9300 2550
+	1    0    0    -1
+$EndComp
+$Comp
+L power:GNDPWR #PWR0104
+U 1 1 5DA502BE
+P 1700 2400
+F 0 "#PWR0104" H 1700 2200 50  0001 C CNN
+F 1 "GNDPWR" H 1704 2246 50  0001 C CNN
+F 2 "" H 1700 2350 50  0001 C CNN
+F 3 "" H 1700 2350 50  0001 C CNN
+	1    1700 2400
+	1    0    0    -1
+$EndComp
+Wire Wire Line
+	1700 2400 1700 2300
+Wire Wire Line
+	1700 2300 1850 2300
+Wire Wire Line
+	1850 2300 1850 2400
 $EndSCHEMATC
