File: preamp-comby/Hierarchy.kicad_pcb (KiCad board)
At the start: 2 copper layers, 64 parts, among them J201 Screw_Terminal_01x03, J301 Tone block On/Off, J302 100k, J303 IN, J304 100k, J305 OUT, J306 9K Filter On/Off, Q201 BD140, Q202 BD139, Q203 2N3904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

Commit message: Finish schematic, start routing
Parts:
- added C201: 5uF, Capacitor_THT:CP_Radial_D5.0mm_P2.00mm, B.Cu at (197.9, 138.5)
- added C202: 5uF, Capacitor_THT:CP_Radial_D5.0mm_P2.00mm, B.Cu at (184.6, 138.5)
- added C203: 120nF, Capacitor_THT:C_Rect_L7.2mm_W3.0mm_P5.00mm_FKS2_FKP2_MKS2_MKP2, B.Cu at (175.4, 139.5)
- added C204: 120n, Capacitor_THT:C_Rect_L7.2mm_W3.0mm_P5.00mm_FKS2_FKP2_MKS2_MKP2, B.Cu at (175.4, 134.9)
- added C205: 5uF, Capacitor_THT:CP_Radial_D5.0mm_P2.00mm, B.Cu at (175.9, 132.2)
- added C206: 5uF, Capacitor_THT:CP_Radial_D5.0mm_P2.00mm, B.Cu at (184.6, 114.2)
- added C207: 5uF, Capacitor_THT:CP_Radial_D5.0mm_P2.00mm, B.Cu at (191.2, 138.5)
- added C208: 5uF, Capacitor_THT:CP_Radial_D5.0mm_P2.00mm, B.Cu at (191.2, 114.2)
- added C301: 0.015u, Capacitor_THT:C_Rect_L7.2mm_W3.0mm_P5.00mm_FKS2_FKP2_MKS2_MKP2, B.Cu at (71.1, 97.1)
- added C302: 0,1u, Capacitor_THT:C_Rect_L7.2mm_W3.0mm_P5.00mm_FKS2_FKP2_MKS2_MKP2, B.Cu at (62.3, 92.5)
- added C303: 0.15u, Capacitor_THT:C_Rect_L7.2mm_W3.0mm_P5.00mm_FKS2_FKP2_MKS2_MKP2, B.Cu at (79.8, 106.2)
- added C304: 0.15u, Capacitor_THT:C_Rect_L7.2mm_W3.0mm_P5.00mm_FKS2_FKP2_MKS2_MKP2, B.Cu at (110.5, 55.8)
- added C305: 3300p, Capacitor_THT:C_Rect_L7.2mm_W3.0mm_P5.00mm_FKS2_FKP2_MKS2_MKP2, B.Cu at (62.3, 97.1)
- added C306: 0.047u, Capacitor_THT:C_Rect_L7.2mm_W3.0mm_P5.00mm_FKS2_FKP2_MKS2_MKP2, B.Cu at (71.1, 106.2)
- added C307: 5u, Capacitor_THT:CP_Radial_D5.0mm_P2.00mm, B.Cu at (80.3, 94.1)
- added C308: 5u, Capacitor_THT:CP_Radial_D5.0mm_P2.00mm, B.Cu at (80.3, 100.6)
- added C309: 0.1u, Capacitor_THT:C_Rect_L7.2mm_W3.0mm_P5.00mm_FKS2_FKP2_MKS2_MKP2, B.Cu at (62.3, 101.6)
- added C310: 0.01u, Capacitor_THT:C_Rect_L7.2mm_W3.0mm_P5.00mm_FKS2_FKP2_MKS2_MKP2, B.Cu at (62.3, 106.2)
- J201, J301, J302, J303, J304, J305, J306, Q201, Q202, Q203, Q204, RV201, RV202, RV301: moved to B.Cu
- moved J201 79.3 mm to (124.3, 128.9)
- moved Q202 75.8 mm to (134.8, 130.0)
- moved Q203 75.8 mm to (147.9, 121.1)
- moved R201 75.8 mm to (140.5, 133.7)
- moved R211 75.8 mm to (155.4, 119.5)
- moved TP203 75.8 mm to (160.5, 129.5)
- moved TP206 75.8 mm to (160.5, 133.0)
- moved D201 75.8 mm to (152.3, 131.9)
- moved D202 75.8 mm to (152.3, 135.2)
- moved Q204 75.8 mm to (133.0, 136.9)
- moved R202 75.8 mm to (145.1, 129.2)
- moved R203 75.8 mm to (151.0, 125.3)
- moved R204 75.8 mm to (140.5, 136.9)
- moved R205 75.8 mm to (151.0, 128.6)
- moved R206 75.8 mm to (146.4, 139.1)
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Connections:
- J201 pad 2: GNDPWR -> GNDA
- R210 pad 2: GNDPWR -> GNDA
- R211 pad 1: GNDPWR -> GNDA
- R321 pad 1: /Preamp/+31V -> /Power/+31V
- R322 pad 1: /Preamp/-31V -> /Power/-31V
Routing:
- net Net-(C309-Pad1): track 0.00 -> 9.91 mm
- net Net-(C307-Pad1): track 0.00 -> 9.04 mm
- net Net-(Q302-Pad3): track 0.00 -> 8.40 mm
- net Net-(Q303-Pad2): track 0.00 -> 8.05 mm
- net Net-(Q301-Pad3): track 0.00 -> 8.02 mm
- net GNDA: track 0.00 -> 5.75 mm
- net Net-(C304-Pad1): track 0.00 -> 4.15 mm
- net Net-(C304-Pad2): track 0.00 -> 3.56 mm
- net Net-(Q302-Pad2): track 0.00 -> 2.76 mm
- net Net-(R312-Pad1): track 0.00 -> 2.18 mm
- net Net-(Q301-Pad2): track 0.00 -> 2.12 mm

Commit message: Routing in progress
Parts:
- moved C309 61.5 mm to (101.9, 54.6), turned to 270 degrees
- moved C307 47.9 mm to (98.8, 49.9)
- moved R318 37.6 mm to (106.7, 60.4), turned to 180 degrees
- moved Q305 26.2 mm to (98.9, 52.4)
- moved Q306 17.7 mm to (102.1, 62.8)
- moved R321 17.2 mm to (89.5, 51.4), turned to 270 degrees
- moved R320 12.4 mm to (99.0, 62.2), turned to 270 degrees
- moved R319 10.2 mm to (99.0, 57.3), turned to 270 degrees
- moved R324 9.91 mm to (90.6, 44.2)
- moved R315 5.70 mm to (113.8, 64.0), turned to 180 degrees
- moved R312 4.48 mm to (106.7, 62.7)
- moved R317 0.99 mm to (105.4, 56.5)
Routing:
- net Net-(C307-Pad1): track 9.04 -> 23.8 mm
- net Net-(C308-Pad2): track 0.00 -> 13.3 mm
- net Net-(C309-Pad2): track 0.00 -> 11.5 mm
- net Net-(C309-Pad1): track 9.91 -> 20.0 mm
- net /Preamp/feedbackTo: track 0.00 -> 8.66 mm
- net Net-(Q305-Pad2): track 0.00 -> 2.89 mm
- net Net-(R312-Pad1): track 2.18 -> 4.79 mm
- net Net-(Q306-Pad2): track 0.00 -> 2.11 mm
- net /Preamp/feedbackFrom: track 0.00 -> 1.90 mm
- net GNDA: track 5.75 -> 4.78 mm
